Commit message: Add files via upload

File: ravens/assets/packOBJ/pack_obj_template.urdf (robot description, URDF)
Before this commit: robot cube.urdf, 1 links, 0 joints
Links:
- link baseLink: geometry collision mesh filename=dataset/our_oriented_decomp/FILENAME.obj scale=.01 .01 .01; visual mesh filename=dataset/our_oriented_dataset/FILENAME.ply scale=.01 .01 .01
